File: encoder-electronics/tc2/kicad/themis_tc2.kicad_pcb (KiCad board)
At the start: 4 copper layers, 99.6 x 99.6 mm, 109 parts, among them J1 Conn_01x02_Pin, J10 Conn_01x02_Pin, J11 Conn_01x02_Pin, J12 Conn_01x08_Pin, J13 Conn_01x02_Pin, J14 Conn_01x03_Pin, J15 Conn_01x02_Pin, J16 Screw_Terminal_01x02, J17 Conn_01x02_Pin, J18 Conn_01x02_Pin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

Commit message: Generate iBOM for TC2
Parts:
- U1: value LT3097ADJC-PBF -> LT3097
- U3, U6: value AD8130ARZ -> AD8130
- U5: value ADS131M03QPWRQ1 -> ADS131M03
